Commit message: URDF updates

File: urdf/blinky.urdf (robot description, URDF)
Before this commit: robot blinky, 7 links, 6 joints
Links:
- added link imu; visual box size=.02 .01 .005
- added link lidar; visual cylinder length=.02 radius=.05
- added link steering_servo; visual box size=.04 .02 .01
- added link steering_servo_arm; visual box size=.005 .005 .015
Joints:
- added joint imu_joint: type fixed, parent base_link, child imu, origin xyz=.16 0 .05
- added joint lidar_joint: type fixed, parent base_link, child lidar, origin xyz=-.06 0 .05
- added joint steering_servo_arm_joing: type revolute, parent steering_servo, child steering_servo_arm, origin xyz=.021 0 .005, limit lower=-0.7854 upper=0.7854 effort=-1 velocity=-1
- added joint steering_servo_joint: type fixed, parent base_link, child steering_servo, origin xyz=.08 0 -.04
- joint front_left_steering_joint: axis 0 0 1 -> 0 0 -1; limit (none) -> lower=-1.57075 upper=1.57075 effort=-1 velocity=-1; type continuous -> revolute
- joint front_right_steering_joint: axis 0 0 1 -> 0 0 -1; limit (none) -> lower=-1.57075 upper=1.57075 effort=-1 velocity=-1; type continuous -> revolute

Commit message: Fix a typo in URDF

File: urdf/blinky.urdf (robot description, URDF)
Before this commit: robot blinky, 11 links, 10 joints
Joints:
- removed joint steering_servo_arm_joing
- added joint steering_servo_arm_joint: type revolute, parent steering_servo, child steering_servo_arm, origin xyz=.021 0 .005, limit lower=-0.7854 upper=0.7854 effort=-1 velocity=-1

Commit message: Add base_footprint to URDF

File: urdf/blinky.urdf (robot description, URDF)
Before this commit: robot blinky, 11 links, 10 joints
Links:
- added link base_footprint
Joints:
- added joint base_link_joint: type fixed, parent base_footprint, child base_link, origin xyz=0 0 .1

Commit message: Fix axis on steering joints

File: urdf/blinky.urdf (robot description, URDF)
Before this commit: robot blinky, 12 links, 11 joints
Joints:
- joint front_left_steering_joint: axis 0 0 -1 -> 0 0 1
- joint front_right_steering_joint: axis 0 0 -1 -> 0 0 1

Commit message: Rotate IMU to be correct

File: urdf/blinky.urdf (robot description, URDF)
Before this commit: robot blinky, 12 links, 11 joints
Joints:
- joint imu_joint: origin xyz=.16 0 .05 -> xyz=.16 0 .05 rpy=3.14159 0 0

Commit message: Add transmissions, remove servo arm

File: urdf/blinky.urdf (robot description, URDF)
Before this commit: robot blinky, 12 links, 11 joints
Links:
- removed link steering_servo_arm
Joints:
- removed joint steering_servo_arm_joint

Commit message: Revert "Rotate IMU to be correct"
This reverts commit bda4b281c780c2f8a5b460ab56b594c3695a26a9.

File: urdf/blinky.urdf (robot description, URDF)
Before this commit: robot blinky, 11 links, 10 joints
Joints:
- joint imu_joint: origin xyz=.16 0 .05 rpy=3.14159 0 0 -> xyz=.16 0 .05
